Commit message: Removed unwanted xacros and updated the URDF file with the correct path to the meshes

File: robot_model/mp_400/mp_400.urdf (robot description, URDF)
Before this commit: robot mp_400, 9 links, 8 joints
Links:
- link base_footprint: geometry collision mesh filename=package://neo_mp_400-2/robot_model/mp_400/meshes/MP-400-BOD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 scale=0.001 0.001 0.001; visual mesh filename=package://neo_mp_400-2/robot_model/mp_400/meshes/MP-400-BOD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 scale=0.001 0.001 0.001
- link lidar_1_link: geometry collision mesh filename=package://neo_mp_400-2/robot_model/mp_400/meshes/SICK-S300.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 scale=0.001 0.001 0.001; visual mesh filename=package://neo_mp_400-2/robot_model/mp_400/meshes/SICK-S300.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 scale=0.001 0.001 0.001
- link mp_400_wheel_back_left_link: geometry collision mesh filename=package://neo_mp_400-2/robot_model/mp_400/meshes/MP-400-CAS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 scale=0.001 0.001 0.001; visual mesh filename=package://neo_mp_400-2/robot_model/mp_400/meshes/MP-400-CAS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 scale=0.001 0.001 0.001
- link mp_400_wheel_back_right_link: geometry collision mesh filename=package://neo_mp_400-2/robot_model/mp_400/meshes/MP-400-CAS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 scale=0.001 0.001 0.001; visual mesh filename=package://neo_mp_400-2/robot_model/mp_400/meshes/MP-400-CAS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 scale=0.001 0.001 0.001
- link mp_400_wheel_front_left_link: geometry collision mesh filename=package://neo_mp_400-2/robot_model/mp_400/meshes/MP-400-CAS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 scale=0.001 0.001 0.001; visual mesh filename=package://neo_mp_400-2/robot_model/mp_400/meshes/MP-400-CAS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 scale=0.001 0.001 0.001
- link mp_400_wheel_front_right_link: geometry collision mesh filename=package://neo_mp_400-2/robot_model/mp_400/meshes/MP-400-CAS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 scale=0.001 0.001 0.001; visual mesh filename=package://neo_mp_400-2/robot_model/mp_400/meshes/MP-400-CAS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 scale=0.001 0.001 0.001
- link mp_400_wheel_left_link: geometry collision mesh filename=package://neo_mp_400-2/robot_model/mp_400/meshes/MP-400-FIX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 scale=0.001 0.001 0.001; visual mesh filename=package://neo_mp_400-2/robot_model/mp_400/meshes/MP-400-FIX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 scale=0.001 0.001 0.001
- link mp_400_wheel_right_link: geometry collision mesh filename=package://neo_mp_400-2/robot_model/mp_400/meshes/MP-400-FIX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 scale=0.001 0.001 0.001; visual mesh filename=package://neo_mp_400-2/robot_model/mp_400/meshes/MP-400-FIX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 scale=0.001 0.001 0.001
