Commit message: adding imu and realsense camera

File: robot_model/mp_400/mp_400.urdf.xacro (robot description, xacro)
@@ -1,24 +1,13 @@
 <?xml version="1.0" ?>
-<!-- =================================================================================== -->
-<!-- |    This document was autogenerated by xacro from mp_400.urdf.xacro              | -->
-<!-- |    EDITING THIS FILE BY HAND IS NOT RECOMMENDED                                 | -->
-<!-- =================================================================================== -->
-<robot name="mp_400">
-  <!--++++++++++++++++++++++++++++++base_link++++++++++++++++++++++++++++++++++++++++++++++++++++-->
-  <!--++++++++++++++++++++body++++++++++++++++++++++++++++-->
+<robot xmlns:xacro="http://www.ros.org/wiki/xacro" name="mp_400">
   <!-- SENSORS -->
-  <!-- Sick S300 - Comment/Uncomment if required  -->
-  <!-- Microscan - Comment/Uncomment if required -->
-  <!-- <xacro:include filename="$(find neo_mp_400-2)/robot_model/mp_400/xacros/micro_scan.xacro" /> -->
-  <!-- Nanoscan - Comment/Uncomment if required -->
-  <!-- <xacro:include filename="$(find neo_mp_400-2)/robot_model/mp_400/xacros/nano_scan.xacro" /> -->
-  <!-- USS and IMU - Comment/Uncomment if required  -->
-  <!-- <xacro:include filename="$(find neo_mp_400-2)/robot_model/mp_400/xacros/imu.xacro" />
-<xacro:include filename="$(find neo_mp_400-2)/robot_model/mp_400/xacros/ultrasonic.xacro" /> -->
+  <xacro:arg name="use_imu" default="false"/>
+  <xacro:arg name="use_d435" default="false"/>
+  <xacro:property name="imu" value="$(arg use_imu)"/>
+  <xacro:property name="d435" value="$(arg use_d435)"/>
   <link name="base_link"/>
   <joint name="base_footprint_joint" type="fixed">
     <origin rpy="0 0 0" xyz="0 0 0"/>
     <axis xyz="0 0 -1"/>
-    <!-- <limit effort="1000.0" lower="-1e+16" upper="1e+16" velocity="3.5"/> -->
     <joint_properties damping="1" friction="1"/>
     <parent link="base_link"/>
@@ -225,9 +214,27 @@
     </collision>
   </link>
-  <!--+++++++++++++++++++ IMU ++++++++++++++++++++++++-->
-  <!-- Comment or uncomment based on your requirement -->
-  <!--   <xacro:imu name="imu_1" parent="base_link">
-    <origin xyz="0.100 0 0.300" rpy="0 0 3.14" />
-  </xacro:imu> -->
+  <!-- Realsense D435 -->
+  <xacro:if value="${d435 == True}">
+    <xacro:include filename="$(find realsense2_description)/urdf/_d435.urdf.xacro"/>
+    <xacro:sensor_d435 parent="base_link">
+      <origin xyz="0.292 0.0 0.716" rpy="0 0 0"/>
+    </xacro:sensor_d435>
+  </xacro:if>
+  <!-- Using IMU -->
+  <xacro:if value="${imu == True}">
+    <link name="imu_link">
+      <inertial>
+        <mass value="0.001" />
+        <origin xyz="0 0 0" rpy="0 0 0" />
+        <inertia ixx="0.0001" ixy="0" ixz="0" iyy="0.000001" iyz="0" izz="0.0001" />
+      </inertial>
+    </link>
+    <joint name="imu2_joint" type="fixed">
+      <axis xyz="0 1 0"/>
+      <origin rpy="0 0 0" xyz="-0.052 0.208 0.266"/>
+      <parent link="base_link"/>
+      <child link="imu_link"/>
+    </joint>
+  </xacro:if>
   <!--+++++++++++++++++++ Ultra Sonic ++++++++++++++++++++++++-->
   <!-- Comment or uncomment based on your requirement -->
@@ -296,7 +303,3 @@
     <origin xyz="0.230 0 0.300" rpy="0 3.14 3.14" />
   </xacro:us_sensor-->
-  <!--Camera  -->
-  <!-- <xacro:camera name="camera" parent="base_link">
-    <origin xyz="0 0 0.38" rpy="0 0 0" />
-  </xacro:camera> -->
 </robot>

Commit message: updating the position of the IMU

File: robot_model/mp_400/mp_400.urdf.xacro (robot description, xacro)
@@ -232,5 +232,5 @@
     <joint name="imu2_joint" type="fixed">
       <axis xyz="0 1 0"/>
-      <origin rpy="0 0 0" xyz="-0.052 0.208 0.266"/>
+      <origin rpy="0 0 0" xyz="0.250 -0.90 0.1525"/>
       <parent link="base_link"/>
       <child link="imu_link"/>

Commit message: fix typo

File: robot_model/mp_400/mp_400.urdf.xacro (robot description, xacro)
@@ -232,5 +232,5 @@
     <joint name="imu2_joint" type="fixed">
       <axis xyz="0 1 0"/>
-      <origin rpy="0 0 0" xyz="0.250 -0.90 0.1525"/>
+      <origin rpy="0 0 0" xyz="0.250 -0.090 0.1525"/>
       <parent link="base_link"/>
       <child link="imu_link"/>

Commit message: adding uss5 sensors

File: robot_model/mp_400/mp_400.urdf.xacro (robot description, xacro)
@@ -4,6 +4,8 @@
   <xacro:arg name="use_imu" default="false"/>
   <xacro:arg name="use_d435" default="false"/>
+  <xacro:arg name="use_uss5" default="false"/>
   <xacro:property name="imu" value="$(arg use_imu)"/>
   <xacro:property name="d435" value="$(arg use_d435)"/>
+  <xacro:property name="uss5" value="$(arg use_uss5)"/>
   <link name="base_link"/>
   <joint name="base_footprint_joint" type="fixed">
@@ -237,69 +239,24 @@
     </joint>
   </xacro:if>
-  <!--+++++++++++++++++++ Ultra Sonic ++++++++++++++++++++++++-->
-  <!-- Comment or uncomment based on your requirement -->
-  <!-- SENSOR 1 -->
-  <!-- xacro:us_sensor name="us_1" parent="base_link">
-    <origin xyz="0.100 0 0.300" rpy="0 3.14 3.14" />
-  </xacro:us_sensor-->
-  <!-- SENSOR 2 -->
-  <!-- xacro:us_sensor name="us_2" parent="base_link">
-    <origin xyz="0.110 0 0.300" rpy="0 3.14 3.14" />
-  </xacro:us_sensor-->
-  <!-- SENSOR 3 -->
-  <!-- xacro:us_sensor name="us_3" parent="base_link">
-    <origin xyz="0.120 0 0.300" rpy="0 3.14 3.14" />
-  </xacro:us_sensor-->
-  <!-- SENSOR 4 -->
-  <!-- xacro:us_sensor name="us_4" parent="base_link">
-    <origin xyz="0.130 0 0.300" rpy="0 3.14 3.14" />
-  </xacro:us_sensor-->
-  <!-- SENSOR 5 -->
-  <!-- xacro:us_sensor name="us_5" parent="base_link">
-    <origin xyz="0.140 0 0.300" rpy="0 3.14 3.14" />
-  </xacro:us_sensor-->
-  <!-- SENSOR 6 -->
-  <!-- xacro:us_sensor name="us_6" parent="base_link">
-    <origin xyz="0.150 0 0.300" rpy="0 3.14 3.14" />
-  </xacro:us_sensor-->
-  <!-- SENSOR 7 -->
-  <!-- xacro:us_sensor name="us_7" parent="base_link">
-    <origin xyz="0.160 0 0.300" rpy="0 3.14 3.14" />
-  </xacro:us_sensor-->
-  <!-- SENSOR 8 -->
-  <!-- xacro:us_sensor name="us_8" parent="base_link">
-    <origin xyz="0.170 0 0.300" rpy="0 3.14 3.14" />
-  </xacro:us_sensor-->
-  <!-- SENSOR 9 -->
-  <!-- xacro:us_sensor name="us_9" parent="base_link">
-    <origin xyz="0.180 0 0.300" rpy="0 3.14 3.14" />
-  </xacro:us_sensor-->
-  <!-- SENSOR 10 -->
-  <!-- xacro:us_sensor name="us_10" parent="base_link">
-    <origin xyz="0.100 0 0.300" rpy="0 3.14 3.14" />
-  </xacro:us_sensor-->
-  <!-- SENSOR 11 -->
-  <!-- xacro:us_sensor name="us_11" parent="base_link">
-    <origin xyz="0.100 0 0.300" rpy="0 3.14 3.14" />
-  </xacro:us_sensor-->
-  <!-- SENSOR 12 -->
-  <!-- xacro:us_sensor name="us_12" parent="base_link">
-    <origin xyz="0.190 0 0.300" rpy="0 3.14 3.14" />
-  </xacro:us_sensor-->
-  <!-- SENSOR 13 -->
-  <!-- xacro:us_sensor name="us_13" parent="base_link">
-    <origin xyz="0.200 0 0.300" rpy="0 3.14 3.14" />
-  </xacro:us_sensor-->
-  <!-- SENSOR 14 -->
-  <!-- xacro:us_sensor name="us_14" parent="base_link">
-    <origin xyz="0.210 0 0.300" rpy="0 3.14 3.14" />
-  </xacro:us_sensor-->
-  <!-- SENSOR 15 -->
-  <!-- xacro:us_sensor name="us_15" parent="base_link">
-    <origin xyz="0.220 0 0.300" rpy="0 3.14 3.14" />
-  </xacro:us_sensor-->
-  <!-- SENSOR 16 -->
-  <!-- xacro:us_sensor name="us_16" parent="base_link">
-    <origin xyz="0.230 0 0.300" rpy="0 3.14 3.14" />
-  </xacro:us_sensor-->
+  <xacro:if value="${uss5 == True}">
+    <xacro:include filename="$(find neo_mp_400-2)/robot_model/mp_400/uss.xacro" />
+    <xacro:us_sensor name="us_1" parent="base_link">
+      <origin xyz="0.266 0.157 0.280" rpy="0 3.14 3.14" />
+    </xacro:us_sensor>
+    <xacro:us_sensor name="us_2" parent="base_link">
+      <origin xyz="0.298 0 0.280" rpy="0 3.14 3.14" />
+    </xacro:us_sensor>
+    <xacro:us_sensor name="us_3" parent="base_link">
+      <origin xyz="0.266 -0.157 0.280" rpy="0 3.14 3.14" />
+    </xacro:us_sensor>
+    <xacro:us_sensor name="us_4" parent="base_link">
+      <origin xyz="-0.266 0.157 0.280" rpy="0 3.14 3.14" />
+    </xacro:us_sensor>
+    <xacro:us_sensor name="us_5" parent="base_link">
+      <origin xyz="-0.298 0 0.280" rpy="0 3.14 3.14" />
+    </xacro:us_sensor>
+    <xacro:us_sensor name="us_6" parent="base_link">
+      <origin xyz="-0.266 -0.157 0.280" rpy="0 3.14 3.14" />
+    </xacro:us_sensor>
+  </xacro:if>
 </robot>

Commit message: updates

File: robot_model/mp_400/mp_400.urdf.xacro (robot description, xacro)
@@ -4,8 +4,8 @@
   <xacro:arg name="use_imu" default="false"/>
   <xacro:arg name="use_d435" default="false"/>
-  <xacro:arg name="use_uss5" default="false"/>
+  <xacro:arg name="use_uss" default="false"/>
   <xacro:property name="imu" value="$(arg use_imu)"/>
   <xacro:property name="d435" value="$(arg use_d435)"/>
-  <xacro:property name="uss5" value="$(arg use_uss5)"/>
+  <xacro:property name="uss" value="$(arg use_uss)"/>
   <link name="base_link"/>
   <joint name="base_footprint_joint" type="fixed">
@@ -239,23 +239,23 @@
     </joint>
   </xacro:if>
-  <xacro:if value="${uss5 == True}">
+  <xacro:if value="${uss == True}">
     <xacro:include filename="$(find neo_mp_400-2)/robot_model/mp_400/uss.xacro" />
     <xacro:us_sensor name="us_1" parent="base_link">
-      <origin xyz="0.266 0.157 0.280" rpy="0 3.14 3.14" />
+      <origin xyz="-0.266 0.157 0.280" rpy="0 0 2.617" />
     </xacro:us_sensor>
     <xacro:us_sensor name="us_2" parent="base_link">
-      <origin xyz="0.298 0 0.280" rpy="0 3.14 3.14" />
+      <origin xyz="-0.298 0 0.280" rpy="0 0 3.14" />
     </xacro:us_sensor>
     <xacro:us_sensor name="us_3" parent="base_link">
-      <origin xyz="0.266 -0.157 0.280" rpy="0 3.14 3.14" />
+      <origin xyz="-0.266 -0.157 0.280" rpy="0 0 3.665" />
     </xacro:us_sensor>
     <xacro:us_sensor name="us_4" parent="base_link">
-      <origin xyz="-0.266 0.157 0.280" rpy="0 3.14 3.14" />
+      <origin xyz="0.266 0.157 0.280" rpy="0 0 0.523" />
     </xacro:us_sensor>
     <xacro:us_sensor name="us_5" parent="base_link">
-      <origin xyz="-0.298 0 0.280" rpy="0 3.14 3.14" />
+      <origin xyz="0.298 0 0.280" rpy="0 0 0" />
     </xacro:us_sensor>
     <xacro:us_sensor name="us_6" parent="base_link">
-      <origin xyz="-0.266 -0.157 0.280" rpy="0 3.14 3.14" />
+      <origin xyz="0.266 -0.157 0.280" rpy="0 0 5.759" />
     </xacro:us_sensor>
   </xacro:if>

Commit message: Adding more sensors (#32)
* adding imu and realsense camera

* updating the launch files

* no need to relay topics

* updating the position of the IMU

* docking launch updates

* adding docking launch

* fix typo

* adding uss5 sensors

* updating the correct directory

* updates

* updating the frame numbers for USboard

File: robot_model/mp_400/mp_400.urdf.xacro (robot description, xacro)
@@ -1,24 +1,15 @@
 <?xml version="1.0" ?>
-<!-- =================================================================================== -->
-<!-- |    This document was autogenerated by xacro from mp_400.urdf.xacro              | -->
-<!-- |    EDITING THIS FILE BY HAND IS NOT RECOMMENDED                                 | -->
-<!-- =================================================================================== -->
-<robot name="mp_400">
-  <!--++++++++++++++++++++++++++++++base_link++++++++++++++++++++++++++++++++++++++++++++++++++++-->
-  <!--++++++++++++++++++++body++++++++++++++++++++++++++++-->
+<robot xmlns:xacro="http://www.ros.org/wiki/xacro" name="mp_400">
   <!-- SENSORS -->
-  <!-- Sick S300 - Comment/Uncomment if required  -->
-  <!-- Microscan - Comment/Uncomment if required -->
-  <!-- <xacro:include filename="$(find neo_mp_400-2)/robot_model/mp_400/xacros/micro_scan.xacro" /> -->
-  <!-- Nanoscan - Comment/Uncomment if required -->
-  <!-- <xacro:include filename="$(find neo_mp_400-2)/robot_model/mp_400/xacros/nano_scan.xacro" /> -->
-  <!-- USS and IMU - Comment/Uncomment if required  -->
-  <!-- <xacro:include filename="$(find neo_mp_400-2)/robot_model/mp_400/xacros/imu.xacro" />
-<xacro:include filename="$(find neo_mp_400-2)/robot_model/mp_400/xacros/ultrasonic.xacro" /> -->
+  <xacro:arg name="use_imu" default="false"/>
+  <xacro:arg name="use_d435" default="false"/>
+  <xacro:arg name="use_uss" default="false"/>
+  <xacro:property name="imu" value="$(arg use_imu)"/>
+  <xacro:property name="d435" value="$(arg use_d435)"/>
+  <xacro:property name="uss" value="$(arg use_uss)"/>
   <link name="base_link"/>
   <joint name="base_footprint_joint" type="fixed">
     <origin rpy="0 0 0" xyz="0 0 0"/>
     <axis xyz="0 0 -1"/>
-    <!-- <limit effort="1000.0" lower="-1e+16" upper="1e+16" velocity="3.5"/> -->
     <joint_properties damping="1" friction="1"/>
     <parent link="base_link"/>
@@ -225,78 +216,47 @@
     </collision>
   </link>
-  <!--+++++++++++++++++++ IMU ++++++++++++++++++++++++-->
-  <!-- Comment or uncomment based on your requirement -->
-  <!--   <xacro:imu name="imu_1" parent="base_link">
-    <origin xyz="0.100 0 0.300" rpy="0 0 3.14" />
-  </xacro:imu> -->
-  <!--+++++++++++++++++++ Ultra Sonic ++++++++++++++++++++++++-->
-  <!-- Comment or uncomment based on your requirement -->
-  <!-- SENSOR 1 -->
-  <!-- xacro:us_sensor name="us_1" parent="base_link">
-    <origin xyz="0.100 0 0.300" rpy="0 3.14 3.14" />
-  </xacro:us_sensor-->
-  <!-- SENSOR 2 -->
-  <!-- xacro:us_sensor name="us_2" parent="base_link">
-    <origin xyz="0.110 0 0.300" rpy="0 3.14 3.14" />
-  </xacro:us_sensor-->
-  <!-- SENSOR 3 -->
-  <!-- xacro:us_sensor name="us_3" parent="base_link">
-    <origin xyz="0.120 0 0.300" rpy="0 3.14 3.14" />
-  </xacro:us_sensor-->
-  <!-- SENSOR 4 -->
-  <!-- xacro:us_sensor name="us_4" parent="base_link">
-    <origin xyz="0.130 0 0.300" rpy="0 3.14 3.14" />
-  </xacro:us_sensor-->
-  <!-- SENSOR 5 -->
-  <!-- xacro:us_sensor name="us_5" parent="base_link">
-    <origin xyz="0.140 0 0.300" rpy="0 3.14 3.14" />
-  </xacro:us_sensor-->
-  <!-- SENSOR 6 -->
-  <!-- xacro:us_sensor name="us_6" parent="base_link">
-    <origin xyz="0.150 0 0.300" rpy="0 3.14 3.14" />
-  </xacro:us_sensor-->
-  <!-- SENSOR 7 -->
-  <!-- xacro:us_sensor name="us_7" parent="base_link">
-    <origin xyz="0.160 0 0.300" rpy="0 3.14 3.14" />
-  </xacro:us_sensor-->
-  <!-- SENSOR 8 -->
-  <!-- xacro:us_sensor name="us_8" parent="base_link">
-    <origin xyz="0.170 0 0.300" rpy="0 3.14 3.14" />
-  </xacro:us_sensor-->
-  <!-- SENSOR 9 -->
-  <!-- xacro:us_sensor name="us_9" parent="base_link">
-    <origin xyz="0.180 0 0.300" rpy="0 3.14 3.14" />
-  </xacro:us_sensor-->
-  <!-- SENSOR 10 -->
-  <!-- xacro:us_sensor name="us_10" parent="base_link">
-    <origin xyz="0.100 0 0.300" rpy="0 3.14 3.14" />
-  </xacro:us_sensor-->
-  <!-- SENSOR 11 -->
-  <!-- xacro:us_sensor name="us_11" parent="base_link">
-    <origin xyz="0.100 0 0.300" rpy="0 3.14 3.14" />
-  </xacro:us_sensor-->
-  <!-- SENSOR 12 -->
-  <!-- xacro:us_sensor name="us_12" parent="base_link">
-    <origin xyz="0.190 0 0.300" rpy="0 3.14 3.14" />
-  </xacro:us_sensor-->
-  <!-- SENSOR 13 -->
-  <!-- xacro:us_sensor name="us_13" parent="base_link">
-    <origin xyz="0.200 0 0.300" rpy="0 3.14 3.14" />
-  </xacro:us_sensor-->
-  <!-- SENSOR 14 -->
-  <!-- xacro:us_sensor name="us_14" parent="base_link">
-    <origin xyz="0.210 0 0.300" rpy="0 3.14 3.14" />
-  </xacro:us_sensor-->
-  <!-- SENSOR 15 -->
-  <!-- xacro:us_sensor name="us_15" parent="base_link">
-    <origin xyz="0.220 0 0.300" rpy="0 3.14 3.14" />
-  </xacro:us_sensor-->
-  <!-- SENSOR 16 -->
-  <!-- xacro:us_sensor name="us_16" parent="base_link">
-    <origin xyz="0.230 0 0.300" rpy="0 3.14 3.14" />
-  </xacro:us_sensor-->
-  <!--Camera  -->
-  <!-- <xacro:camera name="camera" parent="base_link">
-    <origin xyz="0 0 0.38" rpy="0 0 0" />
-  </xacro:camera> -->
+  <!-- Realsense D435 -->
+  <xacro:if value="${d435 == True}">
+    <xacro:include filename="$(find realsense2_description)/urdf/_d435.urdf.xacro"/>
+    <xacro:sensor_d435 parent="base_link">
+      <origin xyz="0.292 0.0 0.716" rpy="0 0 0"/>
+    </xacro:sensor_d435>
+  </xacro:if>
+  <!-- Using IMU -->
+  <xacro:if value="${imu == True}">
+    <link name="imu_link">
+      <inertial>
+        <mass value="0.001" />
+        <origin xyz="0 0 0" rpy="0 0 0" />
+        <inertia ixx="0.0001" ixy="0" ixz="0" iyy="0.000001" iyz="0" izz="0.0001" />
+      </inertial>
+    </link>
+    <joint name="imu2_joint" type="fixed">
+      <axis xyz="0 1 0"/>
+      <origin rpy="0 0 0" xyz="0.250 -0.090 0.1525"/>
+      <parent link="base_link"/>
+      <child link="imu_link"/>
+    </joint>
+  </xacro:if>
+  <xacro:if value="${uss == True}">
+    <xacro:include filename="$(find neo_mp_400-2)/robot_model/mp_400/uss.xacro" />
+    <xacro:us_sensor name="us_1" parent="base_link">
+      <origin xyz="-0.266 0.157 0.280" rpy="0 0 2.617" />
+    </xacro:us_sensor>
+    <xacro:us_sensor name="us_2" parent="base_link">
+      <origin xyz="-0.298 0 0.280" rpy="0 0 3.14" />
+    </xacro:us_sensor>
+    <xacro:us_sensor name="us_3" parent="base_link">
+      <origin xyz="-0.266 -0.157 0.280" rpy="0 0 3.665" />
+    </xacro:us_sensor>
+    <xacro:us_sensor name="us_9" parent="base_link">
+      <origin xyz="0.266 0.157 0.280" rpy="0 0 0.523" />
+    </xacro:us_sensor>
+    <xacro:us_sensor name="us_10" parent="base_link">
+      <origin xyz="0.298 0 0.280" rpy="0 0 0" />
+    </xacro:us_sensor>
+    <xacro:us_sensor name="us_11" parent="base_link">
+      <origin xyz="0.266 -0.157 0.280" rpy="0 0 5.759" />
+    </xacro:us_sensor>
+  </xacro:if>
 </robot>
