Commit message: making xacros even more simpler

File: robot_model/mp_400/mp_400.urdf.xacro (robot description, xacro)
@@ -22,5 +22,5 @@
       <inertia ixx="1.71402" ixy="0.0" ixz="0.0" iyy="0.8856" iyz="0.0" izz="2.5725"/>
     </inertial>
-    <visual name="body">
+    <visual>
       <origin rpy="0 0 1.57" xyz="0.0 0.0 0."/>
       <geometry>
@@ -35,5 +35,5 @@
     </collision>
   </link>
-  <joint name="mp_400_wheel_front_left_joint" type="fixed">
+  <joint name="caster_wheel_left_joint" type="fixed">
     <origin rpy="0 0 1.57" xyz="0.165 0.155 0.036"/>
     <axis xyz="-1 0 0"/>
@@ -41,25 +41,25 @@
     <limit effort="1000.0" lower="-1e+16" upper="1e+16" velocity="3.5"/>
     <parent link="base_footprint"/>
-    <child link="mp_400_wheel_front_left_link"/>
-  </joint>
-  <link name="mp_400_wheel_front_left_link" type="wheel">
-    <inertial>
-      <mass value="1.4"/>
-      <inertia ixx="0.00499743171" ixy="0.00000004464" ixz="-0.00000002245" iyy="0.00499741733" iyz="-0.00000000164" izz="0.00839239692"/>
-    </inertial>
-    <visual name="caster_wheel">
-      <origin rpy="0 0 0" xyz="0 0 0"/>
-      <geometry>
-        <mesh filename="package://neo_mp_400-2/robot_model/mp_400/meshes/MP-400-CASTER-WHEEL.dae" scale="0.001 0.001 0.001"/>
-      </geometry>
-    </visual>
-    <collision>
-      <origin rpy="0 0 0" xyz="0 0. 0"/>
-      <geometry>
-        <mesh filename="package://neo_mp_400-2/robot_model/mp_400/meshes/MP-400-CASTER-WHEEL.dae" scale="0.001 0.001 0.001"/>
-      </geometry>
-    </collision>
-  </link>
-  <joint name="mp_400_wheel_back_left_joint" type="fixed">
+    <child link="caster_wheel_front_left_link"/>
+  </joint>
+  <link name="caster_wheel_front_left_link">
+    <inertial>
+      <mass value="1.4"/>
+      <inertia ixx="0.00499743171" ixy="0.00000004464" ixz="-0.00000002245" iyy="0.00499741733" iyz="-0.00000000164" izz="0.00839239692"/>
+    </inertial>
+    <visual>
+      <origin rpy="0 0 0" xyz="0 0 0"/>
+      <geometry>
+        <mesh filename="package://neo_mp_400-2/robot_model/mp_400/meshes/MP-400-CASTER-WHEEL.dae" scale="0.001 0.001 0.001"/>
+      </geometry>
+    </visual>
+    <collision>
+      <origin rpy="0 0 0" xyz="0 0. 0"/>
+      <geometry>
+        <mesh filename="package://neo_mp_400-2/robot_model/mp_400/meshes/MP-400-CASTER-WHEEL.dae" scale="0.001 0.001 0.001"/>
+      </geometry>
+    </collision>
+  </link>
+  <joint name="caster_wheel_back_left_joint" type="fixed">
     <origin rpy="0 0 1.57" xyz="-0.220 0.155 0.036"/>
     <axis xyz="-1 0 0"/>
@@ -67,25 +67,25 @@
     <limit effort="1000.0" lower="-1e+16" upper="1e+16" velocity="3.5"/>
     <parent link="base_footprint"/>
-    <child link="mp_400_wheel_back_left_link"/>
-  </joint>
-  <link name="mp_400_wheel_back_left_link" type="wheel">
-    <inertial>
-      <mass value="1.4"/>
-      <inertia ixx="0.00499743171" ixy="0.00000004464" ixz="-0.00000002245" iyy="0.00499741733" iyz="-0.00000000164" izz="0.00839239692"/>
-    </inertial>
-    <visual name="caster_wheel">
-      <origin rpy="0 0 0" xyz="0 0 0"/>
-      <geometry>
-        <mesh filename="package://neo_mp_400-2/robot_model/mp_400/meshes/MP-400-CASTER-WHEEL.dae" scale="0.001 0.001 0.001"/>
-      </geometry>
-    </visual>
-    <collision>
-      <origin rpy="0 0 0" xyz="0 0. 0"/>
-      <geometry>
-        <mesh filename="package://neo_mp_400-2/robot_model/mp_400/meshes/MP-400-CASTER-WHEEL.dae" scale="0.001 0.001 0.001"/>
-      </geometry>
-    </collision>
-  </link>
-  <joint name="mp_400_wheel_front_right_joint" type="fixed">
+    <child link="caster_wheel_back_left_link"/>
+  </joint>
+  <link name="caster_wheel_back_left_link">
+    <inertial>
+      <mass value="1.4"/>
+      <inertia ixx="0.00499743171" ixy="0.00000004464" ixz="-0.00000002245" iyy="0.00499741733" iyz="-0.00000000164" izz="0.00839239692"/>
+    </inertial>
+    <visual>
+      <origin rpy="0 0 0" xyz="0 0 0"/>
+      <geometry>
+        <mesh filename="package://neo_mp_400-2/robot_model/mp_400/meshes/MP-400-CASTER-WHEEL.dae" scale="0.001 0.001 0.001"/>
+      </geometry>
+    </visual>
+    <collision>
+      <origin rpy="0 0 0" xyz="0 0. 0"/>
+      <geometry>
+        <mesh filename="package://neo_mp_400-2/robot_model/mp_400/meshes/MP-400-CASTER-WHEEL.dae" scale="0.001 0.001 0.001"/>
+      </geometry>
+    </collision>
+  </link>
+  <joint name="caster_wheel_front_right_joint" type="fixed">
     <origin rpy="0 0 1.57" xyz="0.165 -0.155 0.036"/>
     <axis xyz="-1 0 0"/>
@@ -93,25 +93,25 @@
     <limit effort="1000.0" lower="-1e+16" upper="1e+16" velocity="3.5"/>
     <parent link="base_footprint"/>
-    <child link="mp_400_wheel_front_right_link"/>
-  </joint>
-  <link name="mp_400_wheel_front_right_link" type="wheel">
-    <inertial>
-      <mass value="1.4"/>
-      <inertia ixx="0.00499743171" ixy="0.00000004464" ixz="-0.00000002245" iyy="0.00499741733" iyz="-0.00000000164" izz="0.00839239692"/>
-    </inertial>
-    <visual name="caster_wheel">
-      <origin rpy="0 0 0" xyz="0 0 0"/>
-      <geometry>
-        <mesh filename="package://neo_mp_400-2/robot_model/mp_400/meshes/MP-400-CASTER-WHEEL.dae" scale="0.001 0.001 0.001"/>
-      </geometry>
-    </visual>
-    <collision>
-      <origin rpy="0 0 0" xyz="0 0. 0"/>
-      <geometry>
-        <mesh filename="package://neo_mp_400-2/robot_model/mp_400/meshes/MP-400-CASTER-WHEEL.dae" scale="0.001 0.001 0.001"/>
-      </geometry>
-    </collision>
-  </link>
-  <joint name="mp_400_wheel_back_right_joint" type="fixed">
+    <child link="caster_wheel_front_right_link"/>
+  </joint>
+  <link name="caster_wheel_front_right_link">
+    <inertial>
+      <mass value="1.4"/>
+      <inertia ixx="0.00499743171" ixy="0.00000004464" ixz="-0.00000002245" iyy="0.00499741733" iyz="-0.00000000164" izz="0.00839239692"/>
+    </inertial>
+    <visual>
+      <origin rpy="0 0 0" xyz="0 0 0"/>
+      <geometry>
+        <mesh filename="package://neo_mp_400-2/robot_model/mp_400/meshes/MP-400-CASTER-WHEEL.dae" scale="0.001 0.001 0.001"/>
+      </geometry>
+    </visual>
+    <collision>
+      <origin rpy="0 0 0" xyz="0 0. 0"/>
+      <geometry>
+        <mesh filename="package://neo_mp_400-2/robot_model/mp_400/meshes/MP-400-CASTER-WHEEL.dae" scale="0.001 0.001 0.001"/>
+      </geometry>
+    </collision>
+  </link>
+  <joint name="caster_wheel_back_right_joint" type="fixed">
     <origin rpy="0 0 1.57" xyz="-0.220 -0.155 0.036"/>
     <axis xyz="-1 0 0"/>
@@ -119,25 +119,25 @@
     <limit effort="1000.0" lower="-1e+16" upper="1e+16" velocity="3.5"/>
     <parent link="base_footprint"/>
-    <child link="mp_400_wheel_back_right_link"/>
-  </joint>
-  <link name="mp_400_wheel_back_right_link" type="wheel">
-    <inertial>
-      <mass value="1.4"/>
-      <inertia ixx="0.00499743171" ixy="0.00000004464" ixz="-0.00000002245" iyy="0.00499741733" iyz="-0.00000000164" izz="0.00839239692"/>
-    </inertial>
-    <visual name="caster_wheel">
-      <origin rpy="0 0 0" xyz="0 0 0"/>
-      <geometry>
-        <mesh filename="package://neo_mp_400-2/robot_model/mp_400/meshes/MP-400-CASTER-WHEEL.dae" scale="0.001 0.001 0.001"/>
-      </geometry>
-    </visual>
-    <collision>
-      <origin rpy="0 0 0" xyz="0 0. 0"/>
-      <geometry>
-        <mesh filename="package://neo_mp_400-2/robot_model/mp_400/meshes/MP-400-CASTER-WHEEL.dae" scale="0.001 0.001 0.001"/>
-      </geometry>
-    </collision>
-  </link>
-  <joint name="mp_400_wheel_right_joint" type="fixed">
+    <child link="caster_wheel_back_right_link"/>
+  </joint>
+  <link name="caster_wheel_back_right_link">
+    <inertial>
+      <mass value="1.4"/>
+      <inertia ixx="0.00499743171" ixy="0.00000004464" ixz="-0.00000002245" iyy="0.00499741733" iyz="-0.00000000164" izz="0.00839239692"/>
+    </inertial>
+    <visual>
+      <origin rpy="0 0 0" xyz="0 0 0"/>
+      <geometry>
+        <mesh filename="package://neo_mp_400-2/robot_model/mp_400/meshes/MP-400-CASTER-WHEEL.dae" scale="0.001 0.001 0.001"/>
+      </geometry>
+    </visual>
+    <collision>
+      <origin rpy="0 0 0" xyz="0 0. 0"/>
+      <geometry>
+        <mesh filename="package://neo_mp_400-2/robot_model/mp_400/meshes/MP-400-CASTER-WHEEL.dae" scale="0.001 0.001 0.001"/>
+      </geometry>
+    </collision>
+  </link>
+  <joint name="wheel_right_joint" type="revolute">
     <origin rpy="0 0 1.57" xyz="0. -0.26 0.074"/>
     <axis xyz="1 0 0"/>
@@ -145,12 +145,12 @@
     <joint_properties damping="1.0" friction="1"/>
     <parent link="base_footprint"/>
-    <child link="mp_400_wheel_right_link"/>
-  </joint>
-  <link name="mp_400_wheel_right_link" type="wheel">
+    <child link="wheel_right_link"/>
+  </joint>
+  <link name="wheel_right_link">
     <inertial>
       <mass value="1.82362"/>
       <inertia ixx="0.00399743171" ixy="0.00000004464" ixz="-0.00000002245" iyy="0.00399741733" iyz="-0.00000000164" izz="0.00739239692"/>
     </inertial>
-    <visual name="fixed_wheel_right">
+    <visual>
       <origin rpy="0 0 3.14" xyz="0 0 0.0"/>
       <geometry>
@@ -165,5 +165,5 @@
     </collision>
   </link>
-  <joint name="mp_400_wheel_left_joint" type="fixed">
+  <joint name="wheel_left_joint" type="revolute">
     <origin rpy="0 0 1.57" xyz="-0. 0.26 0.074"/>
     <axis xyz="1 0 0"/>
@@ -171,12 +171,12 @@
     <joint_properties damping="1.0" friction="1"/>
     <parent link="base_footprint"/>
-    <child link="mp_400_wheel_left_link"/>
-  </joint>
-  <link name="mp_400_wheel_left_link" type="wheel">
+    <child link="wheel_left_link"/>
+  </joint>
+  <link name="wheel_left_link">
     <inertial>
       <mass value="1.82362"/>
       <inertia ixx="0.00399743171" ixy="0.00000004464" ixz="-0.00000002245" iyy="0.00399741733" iyz="-0.00000000164" izz="0.00739239692"/>
     </inertial>
-    <visual name="fixed_wheel_left">
+    <visual>
       <origin rpy="0 0 0" xyz="0 0 0.0"/>
       <geometry>
@@ -197,5 +197,5 @@
     <child link="lidar_1_link"/>
   </joint>
-  <link name="lidar_1_link" type="laser">
+  <link name="lidar_1_link">
     <inertial>
       <mass value="0.001"/>
