Commit message: Completed migration to modern gazebo, reafactore launch files, modularized and restructured urdf

File: robot_model/xacros/uss.xacro (robot description, xacro)
@@ -1,4 +1,9 @@
 <?xml version="1.0"?>
+<!--
+Author: Pradheep Padmanabhan
+Contributor: Adarsh Karan K P
+-->
 <robot xmlns:xacro="http://www.ros.org/wiki/xacro" name="mp_400">
+  <!--Ultrasonic Sensor Macro-->
   <xacro:macro name="us_sensor" params="name parent *origin">
     <joint name="${name}_joint" type="fixed">
@@ -12,5 +17,12 @@
         <mass value="0.001" />
         <origin xyz="0 0 0" rpy="0 0 0" />
-        <inertia ixx="0.0001" ixy="0" ixz="0" iyy="0.000001" iyz="0" izz="0.0001" />
+        <inertia
+          ixx="0.0001"
+          ixy="0"
+          ixz="0"
+          iyy="0.000001"
+          iyz="0"
+          izz="0.0001"
+          />
       </inertial>
     </link>
